Commit message: Fix camera orientation

File: turtlebot3_gazebo/urdf/turtlebot3_waffle.gazebo.xacro (robot description, xacro)
@@ -45,5 +45,5 @@
     <material>Gazebo/FlatBlack</material>
   </gazebo>
-  <!-- <gazebo reference="imu_link">
+  <gazebo reference="imu_link">
     <sensor type="imu" name="imu">
       <always_on>true</always_on>
@@ -51,5 +51,5 @@
     </sensor>
     <material>Gazebo/Grey</material>
-  </gazebo> -->
+  </gazebo>
   <gazebo>
     <plugin name="turtlebot3_waffle_controller" filename="libgazebo_ros_diff_drive.so">
@@ -74,5 +74,4 @@
     </plugin>
   </gazebo>
-<!--
   <gazebo>
     <plugin name="imu_plugin" filename="libgazebo_ros_imu.so">
@@ -102,6 +101,6 @@
       </imu>
     </plugin>
-  </gazebo> -->
-  <!-- <gazebo reference="base_scan">
+  </gazebo>
+  <gazebo reference="base_scan">
     <material>Gazebo/FlatBlack</material>
     <sensor type="ray" name="lds_lfcd_sensor">
@@ -134,5 +133,5 @@
       </plugin>
     </sensor>
-  </gazebo> -->
+  </gazebo>
   <!-- <gazebo reference="camera_rgb_frame">
     <sensor type="depth" name="realsense_R200">
@@ -177,11 +176,10 @@
       </plugin>
     </sensor>
-  </gazebo> -->
+  </gazebohttps://github.com/Mettikodeva/turtlebot3_line_followerhttps://github.com/Mettikodeva/turtlebot3_line_followerhttps://github.com/Mettikodeva/turtlebot3_line_followerhttps://github.com/Mettikodeva/turtlebot3_line_follower> -->
 <!-- camera -->
   <gazebo reference="camera_link">
     <sensor name="camera" type="camera" >
-      <pose>0 0 0.05 0 1.37079 0</pose>
       <always_on>true</always_on>
-      <update_rate>60</update_rate>
+      <update_rate>30</update_rate>
       <visualize>true</visualize>
       <camera>
@@ -196,10 +194,13 @@
         </clip>
       </camera>
-      <save enabled="true">
+      <!-- <save enabled="true">
         <path>/tmp/camera_save</path>
-      </save>
+      </save> -->
+      <!-- <always_on>true</always_on>
+      <update_rate>60</update_rate>
+      <visualize>true</visualize> -->
       <plugin name="camera_controller" filename="libgazebo_ros_camera.so">
         <always_on>true</always_on>
-        <update_rate>60</update_rate>
+        <update_rate>30</update_rate>
         <cameraName>camera</cameraName>
         <imageTopicName>image_raw</imageTopicName>

File: turtlebot3_gazebo/urdf/turtlebot3_waffle.urdf.xacro (robot description, xacro)
@@ -168,5 +168,5 @@
     <parent link="base_link"/>
     <child link="camera_link"/>
-    <origin xyz="0.13 0 0.05" rpy="0 0 0"/>
+    <origin xyz="0.13 0 0.1" rpy="0  1.37079 0"/>
     <child>camera_link</child>
     <parent>base_link</parent>
@@ -174,5 +174,5 @@
   <!-- Down facing camera -->
   <link name="camera_link">
-    <origin xyz="0 0 0" rpy="0 0 0"/>
+    <!-- <origin xyz="0 0 0" rpy="0  1.37079 0"/> -->
     <!-- <pose>0 0 0.075 0 0 0 </pose> -->
     <inertial>
